File: electrical/bridge/host.sch (KiCad schematic (older format))
At the start: 21 parts, among them J2 USB_A, P4 ~rst~, P5 bootldr, P6 swd, U3 crystal-4pin

Commit message: Saved project.
Parts:
- added CR?: STM32F105R8T6, LQFP-64, symbol STM32F105R8T6
Other:
- moved on the sheet: C11, C12, C13, C14, C15, C16, C17, C18, C19, J2, P4, P5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
