File: electrical/bridge/bridge.sch (KiCad schematic (older format))
At the start: 27 parts, among them J1 USB_OTG, P1 ~rst~, P2 bootldr, P3 swd, U1 crystal-4pin, U2 my-NCP1117ST50T3G

Commit message: a
Parts:
- added U? (x2): stm32f405rgt6, LQFP-64, symbol stm32f405rgt6
Other:
- moved on the sheet: C1, C10, C2, C3, C4, C5, C6, C7, C8, C9, D1, D2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

Commit message: Making a schematic.
Parts:
- removed P3: swd, Pin_Headers:Pin_Header_Straight_1x03, symbol CONN_01X03
- removed R5: 10k 5%, Resistors_SMD:R_0805, symbol R
- removed R7, R8: 33 5%, Resistors_SMD:R_0805, symbol R
- removed stm1: STM32F103CBT6, my-lib:LQFP48, symbol STM32F103CBT6
- added C? (x2): 2u2, symbol C
- added C?: 100n, Capacitors_SMD:C_0805, symbol C
- added C?: 4u7, Capacitors_SMD:C_0805, symbol C
- added J?: USB_A, symbol USB_A
Connections:
- net labels added: dev_dm, dev_dp, host_dm, host_dp, rx, swd_clk, swd_io, tx
- net labels removed: boot1, d+, d-, rxd, swd-clk, swd-io, txd
- wire segments 87 -> 99
- no-connect marks 4 -> 21
Other:
- note added: "Host"
- note added: "Low speed: 1.5 Mb/s\nFull speed: 12 Mb/s\nHigh speed: 480 Mb/s"
- moved on the sheet: C1, C10, C2, C3, C4, C5, C6, C7, C8, C9, D1, D2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

Commit message: Designing schematic.
Parts:
- removed P1: ~rst~, Measurement_Points:Measurement_Point_Round-TH_Small, symbol CONN_01X01
- added J?: swd, symbol CONN_01X03
- added P?: ~rst~, Pin_Headers:Pin_Header_Straight_1x02, symbol CONN_01X02
Connections:
- wire segments 99 -> 105
- no-connect marks 21 -> 40
Changed lines of the file:
@@
-$EndComp
-$Comp
-L CONN_01X01 P1
-U 1 1 5A699B9E
-P 1375 12475
-F 0 "P1" H 1375 12575 50  0000 C CNN
-F 1 "~rst~" V 1475 12475 50  0000 C CNN
-F 2 "Measurement_Points:Measurement_Point_Round-TH_Small" H 1375 12475 60  0001 C CNN
-F 3 "" H 1375 12475 60  0000 C CNN
-	1    1375 12475
-	-1   0    0    1
 $EndComp
 $Comp
@@
 NoConn ~ 13350 6850
 NoConn ~ 13350 7050
+NoConn ~ 13350 7250
+NoConn ~ 13350 7450
+NoConn ~ 13350 7650
+NoConn ~ 13350 7850
+NoConn ~ 13350 8050
+NoConn ~ 13350 8250
+NoConn ~ 13350 8450
+NoConn ~ 16750 2850
+NoConn ~ 16750 3450
+NoConn ~ 16750 3650
+NoConn ~ 16750 3850
+NoConn ~ 16750 4050
+NoConn ~ 16750 4250
+NoConn ~ 16750 4450
+NoConn ~ 16750 4650
+NoConn ~ 16750 4850
+NoConn ~ 16750 5050
+NoConn ~ 16750 5250
+NoConn ~ 16750 5850
+$Comp
+L CONN_01X03 J?
+U 1 1 5A6E9FA9
+P 18200 3050
+F 0 "J?" H 18200 3250 50  0000 C CNN
+F 1 "swd" V 18300 3050 50  0000 C CNN
+F 2 "" H 18200 3050 50  0001 C CNN
+F 3 "" H 18200 3050 50  0001 C CNN
+	1    18200 3050
+	1    0    0    -1
+$EndComp
+Wire Wire Line
+	17625 2950 18000 2950
+Wire Wire Line
+	17625 3150 18000 3150
+Wire Wire Line
+	18000 3050 17500 3050
+Wire Wire Line
+	17500 3050 17500 3250
+$Comp
+L GND #PWR?
+U 1 1 5A6EA3AE
+P 17500 3250
+F 0 "#PWR?" H 17500 3000 50  0001 C CNN
+F 1 "GND" H 17500 3100 50  0000 C CNN
+F 2 "" H 17500 3250 60  0000 C CNN
+F 3 "" H 17500 3250 60  0000 C CNN
+	1    17500 3250
+	-1   0    0    -1
+$EndComp
+Text Label 17650 2950 0    60   ~ 0
+swd_clk
+Text Label 17650 3150 0    60   ~ 0
+swd_io
+$Comp
+L CONN_01X02 P?
+U 1 1 5A6EB4A8
+P 1375 12525
+F 0 "P?" H 1375 12675 50  0000 C CNN
+F 1 "~rst~" V 1475 12525 50  0000 C CNN
+F 2 "Pin_Headers:Pin_Header_Straight_1x02" H 1375 12525 60  0001 C CNN
+F 3 "" H 1375 12525 60  0000 C CNN
+	1    1375 12525
+	-1   0    0    -1
+$EndComp
+Wire Wire Line
+	1575 12575 1675 12575
+Wire Wire Line
+	1675 12575 1675 12675
+$Comp
+L GND #PWR?
+U 1 1 5A6EB7C8
+P 1675 12675
+F 0 "#PWR?" H 1675 12425 50  0001 C CNN
+F 1 "GND" H 1675 12525 50  0000 C CNN
+F 2 "" H 1675 12675 60  0000 C CNN
+F 3 "" H 1675 12675 60  0000 C CNN
+	1    1675 12675
+	1    0    0    -1
+$EndComp
 $EndSCHEMATC

Commit message: a
Parts:
- C1, C4, C5: footprint Capacitors_SMD:C_0805 -> Capacitor_SMD:C_0603_1608Metric
- C10, C11: renamed from C?; footprint (none) -> Capacitor_SMD:C_0603_1608Metric
- C12: renamed from C8; footprint Capacitors_SMD:C_0805 -> Capacitor_SMD:C_0603_1608Metric
- C13: renamed from C9; footprint Capacitors_SMD:C_0805 -> Capacitor_SMD:C_0603_1608Metric
- C14: renamed from C10; footprint Capacitors_SMD:C_0805 -> Capacitor_SMD:C_0603_1608Metric
- C2: renamed from C3; footprint Capacitors_SMD:C_0805 -> Capacitor_SMD:C_0603_1608Metric
- C3: renamed from C2; footprint Capacitors_SMD:C_0805 -> Capacitor_SMD:C_0603_1608Metric
- C6, C9: renamed from C?; footprint Capacitors_SMD:C_0805 -> Capacitor_SMD:C_0603_1608Metric
- C7: renamed from C6; footprint Capacitors_SMD:C_0805 -> Capacitor_SMD:C_0603_1608Metric
- C8: renamed from C7; footprint Capacitors_SMD:C_0805 -> Capacitor_SMD:C_0603_1608Metric
- D1, D2: footprint LEDs:LED-3MM -> LED_THT:LED_D3.0mm
- J1: footprint (none) -> Connector_USB:USB_Micro-B_Molex_47346-0001
- J2: renamed from J?; footprint (none) -> my-lib:my_usb_a
- J3: renamed from J?; footprint (none) -> Connector_PinHeader_1.27mm:PinHeader_1x03_P1.27mm_Vertical
- P1: renamed from P?; footprint Pin_Headers:Pin_Header_Straight_1x02 -> Connector_PinHeader_1.27mm:PinHeader_1x02_P1.27mm_Vertical
- P2: footprint Pin_Headers:Pin_Header_Straight_1x02 -> Connector_PinHeader_1.27mm:PinHeader_1x02_P1.27mm_Vertical
- R1: renamed from R3; footprint Resistors_SMD:R_0805 -> Resistor_SMD:R_0603_1608Metric
- R2: renamed from R6; footprint Resistors_SMD:R_0805 -> Resistor_SMD:R_0603_1608Metric
- R3: renamed from R1; footprint Resistors_SMD:R_0805 -> Resistor_SMD:R_0603_1608Metric
- R4: renamed from R2; footprint Resistors_SMD:R_0805 -> Resistor_SMD:R_0603_1608Metric
- R5: renamed from R4; footprint Resistors_SMD:R_0805 -> Resistor_SMD:R_0603_1608Metric
- U2: renamed from U?; footprint LQFP-64 -> my-lib:stm32f405rgt6
- U3: renamed from U2; footprint TO_SOT_Packages_SMD:SOT-223 -> Package_TO_SOT_SMD:SOT-223
Connections:
- no-connect marks 40 -> 42
Other:
- moved on the sheet: D1, D2

Commit message: Making pcb.
Parts:
- removed C14: 4u7, Capacitor_SMD:C_0603_1608Metric, symbol C
Connections:
- wire segments 105 -> 103
Changed lines of the file:
@@
-$EndComp
-$Comp
-L C C14
-U 1 1 5A699BAB
-P 11925 11950
-F 0 "C14" H 11950 12050 50  0000 L CNN
-F 1 "4u7" H 11950 11850 50  0000 L CNN
-F 2 "Capacitor_SMD:C_0603_1608Metric" H 11963 11800 30  0001 C CNN
-F 3 "" H 11925 11950 60  0000 C CNN
-	1    11925 11950
-	1    0    0    -1
 $EndComp
 $Comp
@@
 	3500 6225 3500 6475
 Wire Wire Line
-	11925 11650 11925 11800
-Wire Wire Line
-	10450 11650 11925 11650
-Wire Wire Line
 	11625 11650 11625 11800
 Wire Wire Line
 	11325 11550 11325 11800
-Connection ~ 11625 11650
 Wire Wire Line
 	11025 11650 11025 11800
@@
 	10725 12100 10725 12250
 Wire Wire Line
-	10450 12250 11925 12250
-Wire Wire Line
 	11025 12250 11025 12100
 Connection ~ 11025 12250
@@
 	11625 12250 11625 12100
 Connection ~ 11325 12250
-Wire Wire Line
-	11925 12250 11925 12100
-Connection ~ 11625 12250
 Wire Notes Line
 	7175 4800 6475 3800
@@
 NoConn ~ 16750 6050
 NoConn ~ 16750 6450
+Wire Wire Line
+	10450 11650 11625 11650
+Wire Wire Line
+	10450 12250 11625 12250
 $EndSCHEMATC
