File: electrical/bridge/bridge.kicad_pcb (KiCad board)
At the start: 2 copper layers, 42.2 x 24.2 mm, 29 parts, among them J1 USB_OTG, J2 USB_A, J3 swd, P1 ~rst~, P2 bootldr, U1 crystal-4pin, U2 stm32f405rgt6, U3 my-NCP1117ST50T3G

Commit message: Making pcb.
Parts:
- removed C14: 4u7, Capacitor_SMD:C_0603_1608Metric
- moved C5 4.96 mm to (171.8, 104.8), turned to 270 degrees
- moved C8 1.58 mm to (156.2, 91.8)
Routing:
- net GND: track 60.6 -> 187.6 mm
- net VDD: track 17.5 -> 100.1 mm, vias 0 -> 5
- net /led-0: track 0.00 -> 6.60 mm
- net /led-1: track 0.00 -> 5.60 mm
- net /~mcu-rst~: track 3.68 -> 6.15 mm
- net Net-(D2-Pad1): track 0.00 -> 2.12 mm
- net Net-(D1-Pad1): track 0.00 -> 2.12 mm
- net /boot0: track 2.22 -> 3.96 mm

Commit message: Done with routing.
Parts:
- moved C2 0.56 mm to (157.5, 99.2)
- moved R2 0.56 mm to (156.0, 99.2)
Routing:
- net /vbus: track 16.1 -> 23.2 mm, vias 1 -> 2
- net GND: track 187.6 -> 180.6 mm
- added copper zone on F.Cu, net GND
- added copper zone on B.Cu, net VDD
