File: electrical/emg/emg.sch (KiCad schematic (older format))
At the start: 64 parts

Commit message: a
Parts:
- removed C?: 2n2, Capacitor_SMD:C_0603_1608Metric, symbol C
- removed C? (x3): 100n, Capacitor_SMD:C_0603_1608Metric, symbol C
- removed C? (x2): 22n, Capacitor_SMD:C_0603_1608Metric, symbol C
- removed R?: 150 1%, Resistor_SMD:R_0603_1608Metric, symbol R
- removed R? (x2): 47k1%, Resistor_SMD:R_0603_1608Metric, symbol R
- removed R? (x4): 10k 1%, Resistor_SMD:R_0603_1608Metric, symbol R
- removed R?: 1k 1%, Resistor_SMD:R_0603_1608Metric, symbol R
- removed R?: 33k 1%, Resistor_SMD:R_0603_1608Metric, symbol R
- removed R? (x2): 1k5 1%, Resistor_SMD:R_0603_1608Metric, symbol R
- removed R? (x2): 1M 1%, Resistor_SMD:R_0603_1608Metric, symbol R
- removed U? (x4): TSZ124IPT, symbol TSZ124IPT
- added C? (x2): 4u7, Capacitor_SMD:C_0603_1608Metric, symbol C
- added C? (x2): 2n2, Capacitor_SMD:C_0603_1608Metric, symbol C
- added C? (x6): 100n, Capacitor_SMD:C_0603_1608Metric, symbol C
- added J? (x7): T3, symbol TEST_1P
- added J?: Ref, symbol TEST_1P
- added R?: 100 5%, Resistor_SMD:R_0603_1608Metric, symbol R
- added R? (x7): 1k 1%, Resistor_SMD:R_0603_1608Metric, symbol R
- added R? (x6): 10k 1%, Resistor_SMD:R_0603_1608Metric, symbol R
- added U? (x6): TSV734IPT, symbol TSV734IPT
- R?: value 33k 1% -> 10k 1%
Connections:
- wire segments 192 -> 222
Other:
- moved on the sheet: C?, R?, U?A, U?B
