File: electrical/emg/emg.sch (KiCad schematic (older format))
At the start: 75 parts, among them J1 USB_B, J10 Ref, J2 swd, J3 T3, J4 T3, J5 T3, J6 T3, J7 T3, J8 T3, J9 T3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

Commit message: a
Parts:
- added R260: 47k1%, Resistor_SMD:R_0603_1608Metric, symbol R
- TP100, TP101, TP102, TP103: footprint (none) -> MountingHole:MountingHole_3.2mm_M3_DIN965_Pad
Connections:
- wire segments 223 -> 225
Changed lines of the file:
@@
 	1    0    0    -1
 $EndComp
-Text GLabel 19450 2250 2    60   Input ~ 0
+Text GLabel 20000 2250 2    60   Input ~ 0
 v_ref
 $Comp
@@
 $EndComp
 Wire Wire Line
-	19125 2250 19450 2250
+	19125 2250 20000 2250
 Wire Wire Line
 	19225 2350 19225 2250
@@
 F 0 "TP100" H 10000 9800 50  0000 C BNN
 F 1 "M3" H 10000 9750 50  0000 C CNN
-F 2 "" H 10000 9500 50  0001 C CNN
+F 2 "MountingHole:MountingHole_3.2mm_M3_DIN965_Pad" H 10000 9500 50  0001 C CNN
 F 3 "" H 10000 9500 50  0001 C CNN
 	1    10000 9500
@@
 $EndComp
 $Comp
-L GND #PWR?
+L GND #PWR048
 U 1 1 5BA50B5E
 P 10000 9700
-F 0 "#PWR?" H 10000 9450 50  0001 C CNN
+F 0 "#PWR048" H 10000 9450 50  0001 C CNN
 F 1 "GND" H 10000 9550 50  0000 C CNN
 F 2 "" H 10000 9700 60  0000 C CNN
@@
 F 0 "TP101" H 10200 9800 50  0000 C BNN
 F 1 "M3" H 10200 9750 50  0000 C CNN
-F 2 "" H 10200 9500 50  0001 C CNN
+F 2 "MountingHole:MountingHole_3.2mm_M3_DIN965_Pad" H 10200 9500 50  0001 C CNN
 F 3 "" H 10200 9500 50  0001 C CNN
 	1    10200 9500
@@
 $EndComp
 $Comp
-L GND #PWR?
+L GND #PWR049
 U 1 1 5BA514E3
 P 10200 9700
-F 0 "#PWR?" H 10200 9450 50  0001 C CNN
+F 0 "#PWR049" H 10200 9450 50  0001 C CNN
 F 1 "GND" H 10200 9550 50  0000 C CNN
 F 2 "" H 10200 9700 60  0000 C CNN
@@
 F 0 "TP102" H 10400 9800 50  0000 C BNN
 F 1 "M3" H 10400 9750 50  0000 C CNN
-F 2 "" H 10400 9500 50  0001 C CNN
+F 2 "MountingHole:MountingHole_3.2mm_M3_DIN965_Pad" H 10400 9500 50  0001 C CNN
 F 3 "" H 10400 9500 50  0001 C CNN
 	1    10400 9500
@@
 $EndComp
 $Comp
-L GND #PWR?
+L GND #PWR050
 U 1 1 5BA516D0
 P 10400 9700
-F 0 "#PWR?" H 10400 9450 50  0001 C CNN
+F 0 "#PWR050" H 10400 9450 50  0001 C CNN
 F 1 "GND" H 10400 9550 50  0000 C CNN
 F 2 "" H 10400 9700 60  0000 C CNN
@@
 F 0 "TP103" H 10600 9800 50  0000 C BNN
 F 1 "M3" H 10600 9750 50  0000 C CNN
-F 2 "" H 10600 9500 50  0001 C CNN
+F 2 "MountingHole:MountingHole_3.2mm_M3_DIN965_Pad" H 10600 9500 50  0001 C CNN
 F 3 "" H 10600 9500 50  0001 C CNN
 	1    10600 9500
@@
 $EndComp
 $Comp
-L GND #PWR?
+L GND #PWR051
 U 1 1 5BA516DD
 P 10600 9700
-F 0 "#PWR?" H 10600 9450 50  0001 C CNN
+F 0 "#PWR051" H 10600 9450 50  0001 C CNN
 F 1 "GND" H 10600 9550 50  0000 C CNN
 F 2 "" H 10600 9700 60  0000 C CNN
@@
 Wire Wire Line
 	10600 9500 10600 9700
+$Comp
+L R R260
+U 1 1 5B9E3524
+P 19700 2525
+F 0 "R260" V 19780 2525 50  0000 C CNN
+F 1 "47k1%" V 19700 2525 50  0000 C CNN
+F 2 "Resistor_SMD:R_0603_1608Metric" V 19630 2525 30  0001 C CNN
+F 3 "" H 19700 2525 30  0000 C CNN
+	1    19700 2525
+	-1   0    0    1
+$EndComp
+Wire Wire Line
+	19700 2250 19700 2375
+Connection ~ 19700 2250
+Wire Wire Line
+	19700 2675 19700 2850
+$Comp
+L GNDA #PWR052
+U 1 1 5B9E3E05
+P 19700 2850
+F 0 "#PWR052" H 19700 2600 50  0001 C CNN
+F 1 "GNDA" H 19700 2700 50  0000 C CNN
+F 2 "" H 19700 2850 50  0001 C CNN
+F 3 "" H 19700 2850 50  0001 C CNN
+	1    19700 2850
+	1    0    0    -1
+$EndComp
 $EndSCHEMATC

Commit message: Making two separate boards. One for ADC and the other one for preamplification.
Parts:
- removed J4, J5, J6, J9: T3, TestPoint:TestPoint_Pad_D1.0mm, symbol TEST_1P
- added J11, J12, J13, J4, J5, J6, J9: Conn_01x05, Pin_Headers:Pin_Header_Straight_1x05_Pitch1.27mm, symbol Conn_01x05
- added J14, J15, J16, J17: T3, TestPoint:TestPoint_Pad_D1.0mm, symbol TEST_1P
- C19: value 100n -> 2n2
- C24: value 2n2 -> 100n
- R17, R18, R19, R20, R21, R22, R23: value 10k 1% -> 1k 1%
Connections:
- net labels added: v_0, v_1, v_2, v_3, v_4, v_5, v_6
- wire segments 225 -> 280
Other:
- moved on the sheet: C25, J10, R25

Commit message: a
Parts:
- added R26, R27, R28, R29, R30, R31, R32: 100k 1%, Resistor_SMD:R_0603_1608Metric, symbol R
Connections:
- wire segments 280 -> 301
Changed lines of the file:
@@
 Text Label 22475 8150 0    60   ~ 0
 v_ref
+$Comp
+L R R26
+U 1 1 5BA0A0A8
+P 17325 3600
+F 0 "R26" V 17405 3600 50  0000 C CNN
+F 1 "100k 1%" V 17325 3600 50  0000 C CNN
+F 2 "Resistor_SMD:R_0603_1608Metric" V 17255 3600 30  0001 C CNN
+F 3 "" H 17325 3600 30  0000 C CNN
+	1    17325 3600
+	0    -1   -1   0
+$EndComp
+Wire Wire Line
+	17475 3600 17575 3600
+Wire Wire Line
+	17575 3600 17575 3925
+Connection ~ 17575 3925
+Wire Wire Line
+	17175 3600 16875 3600
+Text Label 16925 3600 0    60   ~ 0
+v_ref
+$Comp
+L R R27
+U 1 1 5BA0AB2F
+P 17325 5525
+F 0 "R27" V 17405 5525 50  0000 C CNN
+F 1 "100k 1%" V 17325 5525 50  0000 C CNN
+F 2 "Resistor_SMD:R_0603_1608Metric" V 17255 5525 30  0001 C CNN
+F 3 "" H 17325 5525 30  0000 C CNN
+	1    17325 5525
+	0    -1   -1   0
+$EndComp
+Wire Wire Line
+	17175 5525 16875 5525
+Text Label 16925 5525 0    60   ~ 0
+v_ref
+Wire Wire Line
+	17475 5525 17575 5525
+Wire Wire Line
+	17575 5525 17575 5850
+Connection ~ 17575 5850
+$Comp
+L R R28
+U 1 1 5BA0B156
+P 17325 7450
+F 0 "R28" V 17405 7450 50  0000 C CNN
+F 1 "100k 1%" V 17325 7450 50  0000 C CNN
+F 2 "Resistor_SMD:R_0603_1608Metric" V 17255 7450 30  0001 C CNN
+F 3 "" H 17325 7450 30  0000 C CNN
+	1    17325 7450
+	0    -1   -1   0
+$EndComp
+Wire Wire Line
+	17175 7450 16875 7450
+Text Label 16925 7450 0    60   ~ 0
+v_ref
+Wire Wire Line
+	17475 7450 17575 7450
+Wire Wire Line
+	17575 7450 17575 7800
+Connection ~ 17575 7800
+$Comp
+L R R29
+U 1 1 5BA0BAD2
+P 23700 1600
+F 0 "R29" V 23780 1600 50  0000 C CNN
+F 1 "100k 1%" V 23700 1600 50  0000 C CNN
+F 2 "Resistor_SMD:R_0603_1608Metric" V 23630 1600 30  0001 C CNN
+F 3 "" H 23700 1600 30  0000 C CNN
+	1    23700 1600
+	0    -1   -1   0
+$EndComp
+Wire Wire Line
+	23550 1600 23250 1600
+Text Label 23300 1600 0    60   ~ 0
+v_ref
+Wire Wire Line
+	23850 1600 23950 1600
+Wire Wire Line
+	23950 1600 23950 1925
+Connection ~ 23950 1925
+$Comp
+L R R30
+U 1 1 5BA0C1C3
+P 23700 3600
+F 0 "R30" V 23780 3600 50  0000 C CNN
+F 1 "100k 1%" V 23700 3600 50  0000 C CNN
+F 2 "Resistor_SMD:R_0603_1608Metric" V 23630 3600 30  0001 C CNN
+F 3 "" H 23700 3600 30  0000 C CNN
+	1    23700 3600
+	0    -1   -1   0
+$EndComp
+Wire Wire Line
+	23550 3600 23250 3600
+Text Label 23300 3600 0    60   ~ 0
+v_ref
+Wire Wire Line
+	23850 3600 23950 3600
+Wire Wire Line
+	23950 3600 23950 3925
+Connection ~ 23950 3925
+$Comp
+L R R31
+U 1 1 5BA0C8D7
+P 23700 5550
+F 0 "R31" V 23780 5550 50  0000 C CNN
+F 1 "100k 1%" V 23700 5550 50  0000 C CNN
+F 2 "Resistor_SMD:R_0603_1608Metric" V 23630 5550 30  0001 C CNN
+F 3 "" H 23700 5550 30  0000 C CNN
+	1    23700 5550
+	0    -1   -1   0
+$EndComp
+Wire Wire Line
+	23550 5550 23250 5550
+Text Label 23300 5550 0    60   ~ 0
+v_ref
+Wire Wire Line
+	23850 5550 23950 5550
+Wire Wire Line
+	23950 5550 23950 5850
+Connection ~ 23950 5850
+$Comp
+L R R32
+U 1 1 5BA0CF53
+P 23700 7500
+F 0 "R32" V 23780 7500 50  0000 C CNN
+F 1 "100k 1%" V 23700 7500 50  0000 C CNN
+F 2 "Resistor_SMD:R_0603_1608Metric" V 23630 7500 30  0001 C CNN
+F 3 "" H 23700 7500 30  0000 C CNN
+	1    23700 7500
+	0    -1   -1   0
+$EndComp
+Wire Wire Line
+	23550 7500 23250 7500
+Text Label 23300 7500 0    60   ~ 0
+v_ref
+Wire Wire Line
+	23850 7500 23950 7500
+Wire Wire Line
+	23950 7500 23950 7800
+Connection ~ 23950 7800
 $EndSCHEMATC

Commit message: a
Parts:
- added R33, R34, R35, R36, R37, R38, R39: 1k 1%, Resistor_SMD:R_0603_1608Metric, symbol R
Connections:
- wire segments 301 -> 309
Other:
- moved on the sheet: C25, J10, R25
Changed lines of the file:
@@
 	17250 3050 18575 3050
 Wire Wire Line
-	18575 3050 18575 2250
+	18575 3050 18575 1200
 Wire Wire Line
 	18350 2250 18825 2250
@@
 $EndComp
 Wire Wire Line
-	19125 2250 20125 2250
-Wire Wire Line
 	19225 2350 19225 2250
 Connection ~ 19225 2250
@@
 L TEST_1P J10
 U 1 1 5BA28850
-P 20575 2250
-F 0 "J10" H 20575 2520 50  0000 C CNN
-F 1 "Ref" H 20575 2450 50  0000 C CNN
-F 2 "TestPoint:TestPoint_Pad_D2.5mm" H 20775 2250 50  0001 C CNN
-F 3 "" H 20775 2250 50  0001 C CNN
-	1    20575 2250
+P 19300 1200
+F 0 "J10" H 19300 1470 50  0000 C CNN
+F 1 "Ref" H 19300 1400 50  0000 C CNN
+F 2 "TestPoint:TestPoint_Pad_D2.5mm" H 19500 1200 50  0001 C CNN
+F 3 "" H 19500 1200 50  0001 C CNN
+	1    19300 1200
 	0    1    -1   0
 $EndComp
@@
 L R R25
 U 1 1 5BA2AC3E
-P 20275 2250
-F 0 "R25" V 20355 2250 50  0000 C CNN
-F 1 "1k 1%" V 20275 2250 50  0000 C CNN
-F 2 "Resistor_SMD:R_0603_1608Metric" V 20205 2250 30  0001 C CNN
-F 3 "" H 20275 2250 30  0000 C CNN
-	1    20275 2250
+P 19000 1200
+F 0 "R25" V 19080 1200 50  0000 C CNN
+F 1 "1k 1%" V 19000 1200 50  0000 C CNN
+F 2 "Resistor_SMD:R_0603_1608Metric" V 18930 1200 30  0001 C CNN
+F 3 "" H 19000 1200 30  0000 C CNN
+	1    19000 1200
 	0    1    -1   0
 $EndComp
 Wire Wire Line
-	20425 2250 20575 2250
+	19150 1200 19300 1200
 $Comp
 L C C25
 U 1 1 5BA2C690
-P 20500 2500
-F 0 "C25" H 20525 2600 50  0000 L CNN
-F 1 "4u7" H 20525 2400 50  0000 L CNN
-F 2 "Capacitor_SMD:C_0603_1608Metric" H 20538 2350 30  0001 C CNN
-F 3 "" H 20500 2500 60  0000 C CNN
-	1    20500 2500
+P 19225 1450
+F 0 "C25" H 19250 1550 50  0000 L CNN
+F 1 "4u7" H 19250 1350 50  0000 L CNN
+F 2 "Capacitor_SMD:C_0603_1608Metric" H 19263 1300 30  0001 C CNN
+F 3 "" H 19225 1450 60  0000 C CNN
+	1    19225 1450
 	-1   0    0    -1
 $EndComp
 Wire Wire Line
-	20500 2650 20500 2850
+	19225 1600 19225 1800
 $Comp
 L GNDA #PWR042
 U 1 1 5BA2C697
-P 20500 2850
-F 0 "#PWR042" H 20500 2600 50  0001 C CNN
-F 1 "GNDA" H 20500 2700 50  0000 C CNN
-F 2 "" H 20500 2850 50  0001 C CNN
-F 3 "" H 20500 2850 50  0001 C CNN
-	1    20500 2850
+P 19225 1800
+F 0 "#PWR042" H 19225 1550 50  0001 C CNN
+F 1 "GNDA" H 19225 1650 50  0000 C CNN
+F 2 "" H 19225 1800 50  0001 C CNN
+F 3 "" H 19225 1800 50  0001 C CNN
+	1    19225 1800
 	-1   0    0    -1
 $EndComp
 Wire Wire Line
-	20500 2350 20500 2250
-Connection ~ 20500 2250
+	19225 1300 19225 1200
+Connection ~ 19225 1200
 NoConn ~ 9225 3750
 NoConn ~ 9225 3550
@@
 in_6
 NoConn ~ 9225 2750
-Text Label 19175 4075 0    60   ~ 0
+Text Label 19700 4075 0    60   ~ 0
 in_0
 Wire Wire Line
@@
 	1    0    0    -1
 $EndComp
-$Comp
-L GND #PWR044
-U 1 1 5BA50B5E
-P 10000 9700
-F 0 "#PWR044" H 10000 9450 50  0001 C CNN
-F 1 "GND" H 10000 9550 50  0000 C CNN
-F 2 "" H 10000 9700 60  0000 C CNN
-F 3 "" H 10000 9700 60  0000 C CNN
-	1    10000 9700
-	1    0    0    -1
-$EndComp
 Wire Wire Line
 	10000 9500 10000 9700
@@
 	1    0    0    -1
 $EndComp
-$Comp
-L GND #PWR045
-U 1 1 5BA514E3
-P 10200 9700
-F 0 "#PWR045" H 10200 9450 50  0001 C CNN
-F 1 "GND" H 10200 9550 50  0000 C CNN
-F 2 "" H 10200 9700 60  0000 C CNN
-F 3 "" H 10200 9700 60  0000 C CNN
-	1    10200 9700
-	1    0    0    -1
-$EndComp
 Wire Wire Line
 	10200 9500 10200 9700
@@
 	1    0    0    -1
 $EndComp
-$Comp
-L GND #PWR046
-U 1 1 5BA516D0
-P 10400 9700
-F 0 "#PWR046" H 10400 9450 50  0001 C CNN
-F 1 "GND" H 10400 9550 50  0000 C CNN
-F 2 "" H 10400 9700 60  0000 C CNN
-F 3 "" H 10400 9700 60  0000 C CNN
-	1    10400 9700
-	1    0    0    -1
-$EndComp
 Wire Wire Line
 	10400 9500 10400 9700
@@
 F 3 "" H 10600 9500 50  0001 C CNN
 	1    10600 9500
-	1    0    0    -1
-$EndComp
-$Comp
-L GND #PWR047
-U 1 1 5BA516DD
-P 10600 9700
-F 0 "#PWR047" H 10600 9450 50  0001 C CNN
-F 1 "GND" H 10600 9550 50  0000 C CNN
-F 2 "" H 10600 9700 60  0000 C CNN
-F 3 "" H 10600 9700 60  0000 C CNN
-	1    10600 9700
 	1    0    0    -1
 $EndComp
@@
 Wire Wire Line
 	16875 6150 17175 6150
-Text Label 19175 6000 0    60   ~ 0
+Text Label 19700 6000 0    60   ~ 0
 in_1
 Text Label 16925 6150 0    60   ~ 0
@@
 Wire Wire Line
 	16875 8100 17175 8100
-Text Label 19175 7950 0    60   ~ 0
+Text Label 19700 7950 0    60   ~ 0
 in_2
 Text Label 16925 8100 0    60   ~ 0
@@
 Wire Wire Line
 	23250 4225 23550 4225
-Text Label 25550 4075 0    60   ~ 0
+Text Label 26075 4075 0    60   ~ 0
 in_4
 Text Label 23300 4225 0    60   ~ 0
@@
 Wire Wire Line
 	23250 6150 23550 6150
-Text Label 25550 6000 0    60   ~ 0
+Text Label 26075 6000 0    60   ~ 0
 in_5
 Text Label 23300 6150 0    60   ~ 0
@@
 Wire Wire Line
 	23250 8100 23550 8100
-Text Label 25550 7950 0    60   ~ 0
+Text Label 26075 7950 0    60   ~ 0
 in_6
 Text Label 23300 8100 0    60   ~ 0
@@
 Wire Wire Line
 	23250 2225 23550 2225
-Text Label 25550 2075 0    60   ~ 0
+Text Label 26075 2075 0    60   ~ 0
 in_3
 Text Label 23300 2225 0    60   ~ 0
@@
 	23950 7500 23950 7800
 Connection ~ 23950 7800
+$Comp
+L R R33
+U 1 1 5BA1644D
+P 19500 4075
+F 0 "R33" V 19580 4075 50  0000 C CNN
+F 1 "1k 1%" V 19500 4075 50  0000 C CNN
+F 2 "Resistor_SMD:R_0603_1608Metric" V 19430 4075 30  0001 C CNN
+F 3 "" H 19500 4075 30  0000 C CNN
+	1    19500 4075
+	0    -1   -1   0
+$EndComp
+Wire Wire Line
+	19650 4075 19875 4075
+$Comp
+L R R34
+U 1 1 5BA17212
+P 19500 6000
+F 0 "R34" V 19580 6000 50  0000 C CNN
+F 1 "1k 1%" V 19500 6000 50  0000 C CNN
+F 2 "Resistor_SMD:R_0603_1608Metric" V 19430 6000 30  0001 C CNN
+F 3 "" H 19500 6000 30  0000 C CNN
+	1    19500 6000
+	0    -1   -1   0
+$EndComp
+Wire Wire Line
+	19650 6000 19875 6000
+$Comp
+L R R35
+U 1 1 5BA17A20
+P 19500 7950
+F 0 "R35" V 19580 7950 50  0000 C CNN
+F 1 "1k 1%" V 19500 7950 50  0000 C CNN
+F 2 "Resistor_SMD:R_0603_1608Metric" V 19430 7950 30  0001 C CNN
+F 3 "" H 19500 7950 30  0000 C CNN
+	1    19500 7950
+	0    -1   -1   0
+$EndComp
+Wire Wire Line
+	19650 7950 19875 7950
+$Comp
+L R R36
+U 1 1 5BA18493
+P 25875 2075
+F 0 "R36" V 25955 2075 50  0000 C CNN
+F 1 "1k 1%" V 25875 2075 50  0000 C CNN
+F 2 "Resistor_SMD:R_0603_1608Metric" V 25805 2075 30  0001 C CNN
+F 3 "" H 25875 2075 30  0000 C CNN
+	1    25875 2075
+	0    -1   -1   0
+$EndComp
+Wire Wire Line
+	26025 2075 26250 2075
+$Comp
+L R R37
+U 1 1 5BA18B06
+P 25875 4075
+F 0 "R37" V 25955 4075 50  0000 C CNN
+F 1 "1k 1%" V 25875 4075 50  0000 C CNN
+F 2 "Resistor_SMD:R_0603_1608Metric" V 25805 4075 30  0001 C CNN
+F 3 "" H 25875 4075 30  0000 C CNN
+	1    25875 4075
+	0    -1   -1   0
+$EndComp
+Wire Wire Line
+	26025 4075 26250 4075
+$Comp
+L R R38
+U 1 1 5BA19320
+P 25875 6000
+F 0 "R38" V 25955 6000 50  0000 C CNN
+F 1 "1k 1%" V 25875 6000 50  0000 C CNN
+F 2 "Resistor_SMD:R_0603_1608Metric" V 25805 6000 30  0001 C CNN
+F 3 "" H 25875 6000 30  0000 C CNN
+	1    25875 6000
+	0    -1   -1   0
+$EndComp
+Wire Wire Line
+	26025 6000 26250 6000
+$Comp
+L R R39
+U 1 1 5BA19A6B
+P 25875 7950
+F 0 "R39" V 25955 7950 50  0000 C CNN
+F 1 "1k 1%" V 25875 7950 50  0000 C CNN
+F 2 "Resistor_SMD:R_0603_1608Metric" V 25805 7950 30  0001 C CNN
+F 3 "" H 25875 7950 30  0000 C CNN
+	1    25875 7950
+	0    -1   -1   0
+$EndComp
+Wire Wire Line
+	26025 7950 26250 7950
+Wire Wire Line
+	18575 1200 18850 1200
+Wire Wire Line
+	19125 2250 19700 2250
+$Comp
+L GNDA #PWR?
+U 1 1 5BA1C52B
+P 9650 9775
+F 0 "#PWR?" H 9650 9525 50  0001 C CNN
+F 1 "GNDA" H 9650 9625 50  0000 C CNN
+F 2 "" H 9650 9775 50  0001 C CNN
+F 3 "" H 9650 9775 50  0001 C CNN
+	1    9650 9775
+	1    0    0    -1
+$EndComp
 $EndSCHEMATC
