File: electrical/emg/emg.sch (KiCad schematic (older format))
At the start: 97 parts, among them J1 USB_B, J10 Ref, J11 Conn_01x05, J12 Conn_01x05, J13 Conn_01x05, J14 T3, J15 T3, J16 T3, J17 T3, J2 swd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

Commit message: a
Parts:
- added C26: 4u7, Capacitor_SMD:C_0603_1608Metric, symbol C
- R24: value 100 5% -> 10 5%
Connections:
- wire segments 309 -> 310
Changed lines of the file:
@@
 Text Label 2875 20450 1    60   ~ 0
 led-1
-Text Label 8775 4350 0    60   ~ 0
+Text Label 8775 4950 0    60   ~ 0
 led-0
 $Comp
@@
 Connection ~ 2825 3125
 Wire Wire Line
-	8750 4750 9225 4750
+	8750 5350 9225 5350
 Wire Wire Line
 	2375 21000 2375 20800
@@
 	4775 3275 4775 3125
 Connection ~ 4775 3125
-Text Label 8775 4550 0    60   ~ 0
+Text Label 8775 5150 0    60   ~ 0
 led-1
 Wire Wire Line
@@
 Connection ~ 2725 13475
 Wire Wire Line
-	8750 4350 9225 4350
+	8750 4950 9225 4950
 Wire Wire Line
 	12625 1550 13025 1550
@@
 NoConn ~ 9225 3150
 NoConn ~ 9225 3350
-NoConn ~ 9225 4950
-NoConn ~ 9225 5150
-NoConn ~ 9225 5350
+NoConn ~ 9225 4350
+NoConn ~ 9225 4550
+NoConn ~ 9225 4750
 NoConn ~ 9225 5550
 NoConn ~ 9225 5750
@@
 	3800 4600 3475 4600
 Wire Wire Line
-	3475 4600 3475 3125
+	3475 3125 3475 4750
 Connection ~ 3475 3125
 $Comp
@@
 	3375 20250 3375 20500
 Wire Wire Line
-	9225 4550 8750 4550
-Text Label 8775 4750 0    60   ~ 0
+	9225 5150 8750 5150
+Text Label 8775 5350 0    60   ~ 0
 led-2
 $Comp
@@
 P 18975 2250
 F 0 "R24" V 19055 2250 50  0000 C CNN
-F 1 "100 5%" V 18875 2250 50  0000 C CNN
+F 1 "10 5%" V 18875 2250 50  0000 C CNN
 F 2 "Resistor_SMD:R_0603_1608Metric" V 18905 2250 30  0001 C CNN
 F 3 "" H 18975 2250 30  0000 C CNN
@@
 in_6
 NoConn ~ 9225 2750
-Text Label 19700 4075 0    60   ~ 0
+Text Label 19725 7950 0    60   ~ 0
 in_0
 Wire Wire Line
@@
 	19700 2675 19700 2850
 $Comp
-L GNDA #PWR048
+L GNDA #PWR044
 U 1 1 5B9E3E05
 P 19700 2850
-F 0 "#PWR048" H 19700 2600 50  0001 C CNN
+F 0 "#PWR044" H 19700 2600 50  0001 C CNN
 F 1 "GNDA" H 19700 2700 50  0000 C CNN
 F 2 "" H 19700 2850 50  0001 C CNN
@@
 Wire Wire Line
 	17700 3925 16875 3925
-Text Label 16900 3925 0    60   ~ 0
+Text Label 16925 7800 0    60   ~ 0
 v_0
 $Comp
@@
 Wire Wire Line
 	17700 5850 16875 5850
-Text Label 16900 5850 0    60   ~ 0
+Text Label 16925 5850 0    60   ~ 0
 v_1
 $Comp
@@
 Wire Wire Line
 	16875 8100 17175 8100
-Text Label 19700 7950 0    60   ~ 0
+Text Label 19700 4075 0    60   ~ 0
 in_2
 Text Label 16925 8100 0    60   ~ 0
@@
 Wire Wire Line
 	17700 7800 16875 7800
-Text Label 16900 7800 0    60   ~ 0
+Text Label 16925 3925 0    60   ~ 0
 v_2
 $Comp
@@
 	24475 1725 24475 1675
 $Comp
-L VDDA #PWR049
+L VDDA #PWR045
 U 1 1 5BA15A7B
 P 24475 1675
-F 0 "#PWR049" H 24475 1525 50  0001 C CNN
+F 0 "#PWR045" H 24475 1525 50  0001 C CNN
 F 1 "VDDA" H 24475 1825 50  0000 C CNN
 F 2 "" H 24475 1675 50  0001 C CNN
@@
 $EndComp
 $Comp
-L GNDA #PWR050
+L GNDA #PWR046
 U 1 1 5BA163D0
 P 24475 2475
-F 0 "#PWR050" H 24475 2225 50  0001 C CNN
+F 0 "#PWR046" H 24475 2225 50  0001 C CNN
 F 1 "GNDA" H 24475 2325 50  0000 C CNN
 F 2 "" H 24475 2475 50  0001 C CNN
@@
 $EndComp
 $Comp
-L VDDA #PWR051
+L VDDA #PWR047
 U 1 1 5BA17261
 P 22875 1750
-F 0 "#PWR051" H 22875 1600 50  0001 C CNN
+F 0 "#PWR047" H 22875 1600 50  0001 C CNN
 F 1 "VDDA" H 22875 1900 50  0000 C CNN
 F 2 "" H 22875 1750 50  0001 C CNN
@@
 	22875 1925 22875 1750
 $Comp
-L GNDA #PWR052
+L GNDA #PWR048
 U 1 1 5BA17268
 P 22875 2425
-F 0 "#PWR052" H 22875 2175 50  0001 C CNN
+F 0 "#PWR048" H 22875 2175 50  0001 C CNN
 F 1 "GNDA" H 22875 2275 50  0000 C CNN
 F 2 "" H 22875 2425 50  0001 C CNN
@@
 	16100 4025 16100 3975
 $Comp
-L VDDA #PWR053
+L VDDA #PWR049
 U 1 1 5BA19957
 P 16100 3975
-F 0 "#PWR053" H 16100 3825 50  0001 C CNN
+F 0 "#PWR049" H 16100 3825 50  0001 C CNN
 F 1 "VDDA" H 16100 4125 50  0000 C CNN
 F 2 "" H 16100 3975 50  0001 C CNN
@@
 Connection ~ 15725 4225
 $Comp
-L GNDA #PWR054
+L GNDA #PWR050
 U 1 1 5BA1AD6D
 P 15525 4275
-F 0 "#PWR054" H 15525 4025 50  0001 C CNN
+F 0 "#PWR050" H 15525 4025 50  0001 C CNN
 F 1 "GNDA" H 15525 4125 50  0000 C CNN
 F 2 "" H 15525 4275 50  0001 C CNN
@@
 	16175 5875 16175 5825
 $Comp
-L VDDA #PWR055
+L VDDA #PWR051
 U 1 1 5BA1CBB0
 P 16175 5825
-F 0 "#PWR055" H 16175 5675 50  0001 C CNN
+F 0 "#PWR051" H 16175 5675 50  0001 C CNN
 F 1 "VDDA" H 16175 5975 50  0000 C CNN
 F 2 "" H 16175 5825 50  0001 C CNN
@@
 Connection ~ 15800 6075
 $Comp
-L GNDA #PWR056
+L GNDA #PWR052
 U 1 1 5BA1CBBE
 P 15600 6125
-F 0 "#PWR056" H 15600 5875 50  0001 C CNN
+F 0 "#PWR052" H 15600 5875 50  0001 C CNN
 F 1 "GNDA" H 15600 5975 50  0000 C CNN
 F 2 "" H 15600 6125 50  0001 C CNN
@@
 	16200 7725 16200 7675
 $Comp
-L VDDA #PWR057
+L VDDA #PWR053
 U 1 1 5BA1CF9E
 P 16200 7675
-F 0 "#PWR057" H 16200 7525 50  0001 C CNN
+F 0 "#PWR053" H 16200 7525 50  0001 C CNN
 F 1 "VDDA" H 16200 7825 50  0000 C CNN
 F 2 "" H 16200 7675 50  0001 C CNN
@@
 Connection ~ 15825 7925
 $Comp
-L GNDA #PWR058
+L GNDA #PWR054
 U 1 1 5BA1CFAC
 P 15625 7975
-F 0 "#PWR058" H 15625 7725 50  0001 C CNN
+F 0 "#PWR054" H 15625 7725 50  0001 C CNN
 F 1 "GNDA" H 15625 7825 50  0000 C CNN
 F 2 "" H 15625 7975 50  0001 C CNN
@@
 	22275 1875 22275 1825
 $Comp
-L VDDA #PWR059
+L VDDA #PWR055
 U 1 1 5BA1D4BD
 P 22275 1825
-F 0 "#PWR059" H 22275 1675 50  0001 C CNN
+F 0 "#PWR055" H 22275 1675 50  0001 C CNN
 F 1 "VDDA" H 22275 1975 50  0000 C CNN
 F 2 "" H 22275 1825 50  0001 C CNN
@@
 Connection ~ 21900 2075
 $Comp
-L GNDA #PWR060
+L GNDA #PWR056
 U 1 1 5BA1D4CB
 P 21700 2125
-F 0 "#PWR060" H 21700 1875 50  0001 C CNN
+F 0 "#PWR056" H 21700 1875 50  0001 C CNN
 F 1 "GNDA" H 21700 1975 50  0000 C CNN
 F 2 "" H 21700 2125 50  0001 C CNN
@@
 	22450 3875 22450 3825
 $Comp
-L VDDA #PWR061
+L VDDA #PWR057
 U 1 1 5BA1D6ED
 P 22450 3825
-F 0 "#PWR061" H 22450 3675 50  0001 C CNN
+F 0 "#PWR057" H 22450 3675 50  0001 C CNN
 F 1 "VDDA" H 22450 3975 50  0000 C CNN
 F 2 "" H 22450 3825 50  0001 C CNN
@@
 Connection ~ 22075 4075
 $Comp
-L GNDA #PWR062
+L GNDA #PWR058
 U 1 1 5BA1D6FB
 P 21875 4125
-F 0 "#PWR062" H 21875 3875 50  0001 C CNN
+F 0 "#PWR058" H 21875 3875 50  0001 C CNN
 F 1 "GNDA" H 21875 3975 50  0000 C CNN
 F 2 "" H 21875 4125 50  0001 C CNN
@@
 	22500 5800 22500 5750
 $Comp
-L VDDA #PWR063
+L VDDA #PWR059
 U 1 1 5BA1DCCB
 P 22500 5750
-F 0 "#PWR063" H 22500 5600 50  0001 C CNN
+F 0 "#PWR059" H 22500 5600 50  0001 C CNN
 F 1 "VDDA" H 22500 5900 50  0000 C CNN
 F 2 "" H 22500 5750 50  0001 C CNN
@@
 Connection ~ 22125 6000
 $Comp
-L GNDA #PWR064
+L GNDA #PWR060
 U 1 1 5BA1DCD9
 P 21925 6050
-F 0 "#PWR064" H 21925 5800 50  0001 C CNN
+F 0 "#PWR060" H 21925 5800 50  0001 C CNN
 F 1 "GNDA" H 21925 5900 50  0000 C CNN
 F 2 "" H 21925 6050 50  0001 C CNN
@@
 	22625 7750 22625 7700
 $Comp
-L VDDA #PWR065
+L VDDA #PWR061
 U 1 1 5BA1DFD3
 P 22625 7700
-F 0 "#PWR065" H 22625 7550 50  0001 C CNN
+F 0 "#PWR061" H 22625 7550 50  0001 C CNN
 F 1 "VDDA" H 22625 7850 50  0000 C CNN
 F 2 "" H 22625 7700 50  0001 C CNN
@@
 Connection ~ 22250 7950
 $Comp
-L GNDA #PWR066
+L GNDA #PWR062
 U 1 1 5BA1DFE1
 P 22050 8000
-F 0 "#PWR066" H 22050 7750 50  0001 C CNN
+F 0 "#PWR062" H 22050 7750 50  0001 C CNN
 F 1 "GNDA" H 22050 7850 50  0000 C CNN
 F 2 "" H 22050 8000 50  0001 C CNN
@@
 	19125 2250 19700 2250
 $Comp
-L GNDA #PWR?
+L GNDA #PWR063
 U 1 1 5BA1C52B
-P 9650 9775
-F 0 "#PWR?" H 9650 9525 50  0001 C CNN
-F 1 "GNDA" H 9650 9625 50  0000 C CNN
-F 2 "" H 9650 9775 50  0001 C CNN
-F 3 "" H 9650 9775 50  0001 C CNN
-	1    9650 9775
-	1    0    0    -1
-$EndComp
+P 10000 9700
+F 0 "#PWR063" H 10000 9450 50  0001 C CNN
+F 1 "GNDA" H 10000 9550 50  0000 C CNN
+F 2 "" H 10000 9700 50  0001 C CNN
+F 3 "" H 10000 9700 50  0001 C CNN
+	1    10000 9700
+	1    0    0    -1
+$EndComp
+$Comp
+L C C26
+U 1 1 5BA203B3
+P 3475 4900
+F 0 "C26" H 3500 5000 50  0000 L CNN
+F 1 "4u7" H 3500 4800 50  0000 L CNN
+F 2 "Capacitor_SMD:C_0603_1608Metric" H 3513 4750 30  0001 C CNN
+F 3 "" H 3475 4900 60  0000 C CNN
+	1    3475 4900
+	1    0    0    -1
+$EndComp
+Wire Wire Line
+	3475 5050 3475 5150
+Connection ~ 3475 4600
+$Comp
+L GNDA #PWR064
+U 1 1 5BA21351
+P 10200 9700
+F 0 "#PWR064" H 10200 9450 50  0001 C CNN
+F 1 "GNDA" H 10200 9550 50  0000 C CNN
+F 2 "" H 10200 9700 50  0001 C CNN
+F 3 "" H 10200 9700 50  0001 C CNN
+	1    10200 9700
+	1    0    0    -1
+$EndComp
+$Comp
+L GNDA #PWR065
+U 1 1 5BA21497
+P 10400 9700
+F 0 "#PWR065" H 10400 9450 50  0001 C CNN
+F 1 "GNDA" H 10400 9550 50  0000 C CNN
+F 2 "" H 10400 9700 50  0001 C CNN
+F 3 "" H 10400 9700 50  0001 C CNN
+	1    10400 9700
+	1    0    0    -1
+$EndComp
+$Comp
+L GNDA #PWR066
+U 1 1 5BA215DD
+P 10600 9700
+F 0 "#PWR066" H 10600 9450 50  0001 C CNN
+F 1 "GNDA" H 10600 9550 50  0000 C CNN
+F 2 "" H 10600 9700 50  0001 C CNN
+F 3 "" H 10600 9700 50  0001 C CNN
+	1    10600 9700
+	1    0    0    -1
+$EndComp
+$Comp
+L GNDA #PWR067
+U 1 1 5BA227E7
+P 3475 5150
+F 0 "#PWR067" H 3475 4900 50  0001 C CNN
+F 1 "GNDA" H 3475 5000 50  0000 C CNN
+F 2 "" H 3475 5150 50  0001 C CNN
+F 3 "" H 3475 5150 50  0001 C CNN
+	1    3475 5150
+	1    0    0    -1
+$EndComp

Commit message: a
Parts:
- removed J10: Ref, TestPoint:TestPoint_Pad_D2.5mm, symbol TEST_1P
- added J10: Ref, Pin_Headers:Pin_Header_Straight_1x05_Pitch1.27mm, symbol Conn_01x05
Connections:
- wire segments 310 -> 315

Commit message: a
Other:
- note added: "For all opamps no amplification \nto not disturb Vref. \n(Or need to make separate Vref \nsource for each amplifier)"
- note added: "Need to be \nswapped"
Changed lines of the file:
@@
 	19475 1400 19575 1400
 Connection ~ 19475 1300
+Wire Notes Line
+	17175 4100 17475 4350
+Wire Notes Line
+	17250 4375 17425 4100
+Wire Notes Line
+	17150 5975 17500 6300
+Wire Notes Line
+	17175 6325 17425 6000
+Wire Notes Line
+	17225 8350 17450 7875
+Wire Notes Line
+	17200 7900 17475 8350
+Wire Notes Line
+	23600 2125 23825 2375
+Wire Notes Line
+	23600 2350 23825 2100
+Wire Notes Line
+	23550 4475 23825 4000
+Wire Notes Line
+	23500 4025 23825 4450
+Wire Notes Line
+	23600 6000 23850 6325
+Wire Notes Line
+	23600 6325 23800 6000
+Wire Notes Line
+	23550 8275 23800 7900
+Wire Notes Line
+	23575 7925 23825 8275
+Wire Notes Line
+	8600 7150 7500 7875
+Wire Notes Line
+	7500 7875 8675 7375
+Text Notes 7225 8100 0    60   ~ 0
+Need to be \nswapped
+Wire Notes Line
+	17275 8800 17850 11400
+Text Notes 17250 11775 0    60   ~ 0
+For all opamps no amplification \nto not disturb Vref. \n(Or need to make separate Vref \nsource for each amplifier)
 $EndSCHEMATC
