File: electrical/emg/_saved_emg.sch (KiCad schematic (older format))
At the start: 75 parts, among them J1 USB_B, J10 Ref, J2 swd, J3 T3, J4 T3, J5 T3, J6 T3, J7 T3, J8 T3, J9 T3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

Commit message: a
Parts:
- TP100, TP101, TP102, TP103: footprint (none) -> MountingHole:MountingHole_3.2mm_M3_Pad
Changed lines of the file:
@@
 F 0 "TP100" H 10000 9800 50  0000 C BNN
 F 1 "M3" H 10000 9750 50  0000 C CNN
-F 2 "" H 10000 9500 50  0001 C CNN
+F 2 "MountingHole:MountingHole_3.2mm_M3_Pad" H 10000 9500 50  0001 C CNN
 F 3 "" H 10000 9500 50  0001 C CNN
 	1    10000 9500
@@
 $EndComp
 $Comp
-L GND #PWR?
+L GND #PWR048
 U 1 1 5BA50B5E
 P 10000 9700
-F 0 "#PWR?" H 10000 9450 50  0001 C CNN
+F 0 "#PWR048" H 10000 9450 50  0001 C CNN
 F 1 "GND" H 10000 9550 50  0000 C CNN
 F 2 "" H 10000 9700 60  0000 C CNN
@@
 F 0 "TP101" H 10200 9800 50  0000 C BNN
 F 1 "M3" H 10200 9750 50  0000 C CNN
-F 2 "" H 10200 9500 50  0001 C CNN
+F 2 "MountingHole:MountingHole_3.2mm_M3_Pad" H 10200 9500 50  0001 C CNN
 F 3 "" H 10200 9500 50  0001 C CNN
 	1    10200 9500
@@
 $EndComp
 $Comp
-L GND #PWR?
+L GND #PWR049
 U 1 1 5BA514E3
 P 10200 9700
-F 0 "#PWR?" H 10200 9450 50  0001 C CNN
+F 0 "#PWR049" H 10200 9450 50  0001 C CNN
 F 1 "GND" H 10200 9550 50  0000 C CNN
 F 2 "" H 10200 9700 60  0000 C CNN
@@
 F 0 "TP102" H 10400 9800 50  0000 C BNN
 F 1 "M3" H 10400 9750 50  0000 C CNN
-F 2 "" H 10400 9500 50  0001 C CNN
+F 2 "MountingHole:MountingHole_3.2mm_M3_Pad" H 10400 9500 50  0001 C CNN
 F 3 "" H 10400 9500 50  0001 C CNN
 	1    10400 9500
@@
 $EndComp
 $Comp
-L GND #PWR?
+L GND #PWR050
 U 1 1 5BA516D0
 P 10400 9700
-F 0 "#PWR?" H 10400 9450 50  0001 C CNN
+F 0 "#PWR050" H 10400 9450 50  0001 C CNN
 F 1 "GND" H 10400 9550 50  0000 C CNN
 F 2 "" H 10400 9700 60  0000 C CNN
@@
 F 0 "TP103" H 10600 9800 50  0000 C BNN
 F 1 "M3" H 10600 9750 50  0000 C CNN
-F 2 "" H 10600 9500 50  0001 C CNN
+F 2 "MountingHole:MountingHole_3.2mm_M3_Pad" H 10600 9500 50  0001 C CNN
 F 3 "" H 10600 9500 50  0001 C CNN
 	1    10600 9500
@@
 $EndComp
 $Comp
-L GND #PWR?
+L GND #PWR051
 U 1 1 5BA516DD
 P 10600 9700
-F 0 "#PWR?" H 10600 9450 50  0001 C CNN
+F 0 "#PWR051" H 10600 9450 50  0001 C CNN
 F 1 "GND" H 10600 9550 50  0000 C CNN
 F 2 "" H 10600 9700 60  0000 C CNN
