File: electrical/emg/emg.kicad_pcb (KiCad board)
At the start: 2 copper layers, 98 parts, among them J1 USB_B, J10 Ref, J11 Conn_01x05, J12 Conn_01x05, J13 Conn_01x05, J14 T3, J15 T3, J16 T3, J17 T3, J2 swd, J3 T3, J4 Conn_01x05, J5 Conn_01x05, J6 Conn_01x05, J7 T3, J8 T3, J9 Conn_01x05, P1 ~rst~, P2 bootldr, U1 stm32f405rgt6, U2 crystal-4pin, U3 my-NCP1117ST50T3G, U4 my-NCP1117ST50T3G, U5 TSV734IPT, U6 TSV734IPT

Commit message: a
Parts:
- J10: footprint TestPoint:TestPoint_Pad_D2.5mm -> Pin_Headers:Pin_Header_Straight_1x05_Pitch1.27mm
- moved J6 3.85 mm to (151.7, 85.1)
- moved J5 3.15 mm to (148.2, 85.1)
- moved J10 0.87 mm to (131.2, 86.5), turned to 90 degrees
- moved R19 0.20 mm to (142.2, 108.8)
- moved R18 0.05 mm to (142.2, 110.7)
Routing:
- net /v_ref: track 4.53 -> 86.2 mm, vias 0 -> 8
- net GND: track 34.8 -> 104.2 mm
- net GNDA: track 14.3 -> 79.5 mm, vias 2 -> 3
- net VDDA: track 8.74 -> 55.5 mm, vias 2 -> 4
- net /in_4: track 0.00 -> 40.0 mm
- net /in_6: track 0.00 -> 38.8 mm, vias 0 -> 2
- net /in_3: track 0.00 -> 34.4 mm, vias 0 -> 2
- net /in_5: track 0.00 -> 29.8 mm, vias 0 -> 2
- net /v_3: track 4.56 -> 33.3 mm
- net /v_2: track 0.00 -> 27.9 mm, vias 0 -> 2
- net /v_4: track 4.56 -> 29.0 mm
- net /v_5: track 4.59 -> 22.3 mm
- net /v_1: track 4.65 -> 19.8 mm, vias 0 -> 2
- net /v_0: track 4.52 -> 15.3 mm
- net /v_6: track 4.63 -> 13.7 mm
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
Commit message: a
Routing:
- net GNDA: track 79.5 -> 327.0 mm
- net GND: track 104.2 -> 244.4 mm, vias 0 -> 6
- net VDDA: track 55.5 -> 147.9 mm
- net /v_ref: track 86.2 -> 149.2 mm, vias 8 -> 13
- net VDD: track 37.2 -> 98.5 mm, vias 0 -> 4
- net /vbus: track 13.7 -> 29.9 mm, vias 0 -> 1
- net /v_1: track 19.8 -> 22.2 mm
- net /v_2: track 27.9 -> 29.2 mm
Other:
- board outline added: 70 x 37 mm
- copper layers 2 -> 4
