File: electrical/bridge_btns/bridge.kicad_pcb (KiCad board)
At the start: 2 copper layers, 42.2 x 24.2 mm, 43 parts, among them J1 MY_USB_B, J2 MY_USB_B, J3 swd, J4 Conn_01x05, J5 Conn_01x07, J6 Conn_01x14, P1 ~rst~, P2 bootldr, U1 crystal-4pin, U2 stm32f405rgt6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

Commit message: a
Parts:
- removed R17: 0, Resistor_SMD:R_0603_1608Metric
- added J7: Conn_01x14, Connector_PinHeader_1.27mm:PinHeader_1x14_P1.27mm_Vertical, F.Cu at (153.5, 110.5)
- added R18: 10k 5%, Resistor_SMD:R_0603_1608Metric, B.Cu at (157.7, 87.6)
- added R19: 10k 5%, Resistor_SMD:R_0603_1608Metric, B.Cu at (159.4, 87.6)
- C4, C5, C9, R10, R11, R12, R13, R14, R15, R16, R6, R7, R8, R9, U3: moved to B.Cu
- moved J5 37.1 mm to (163.8, 85.3), turned to 90 degrees
- moved J4 36.5 mm to (162.5, 85.3), turned to 270 degrees
- moved C5 22.7 mm to (175.0, 93.5), turned to 0 degrees
- moved R8 22.2 mm to (168.2, 107.1), turned to 90 degrees
- moved R9 22.2 mm to (166.7, 107.1), turned to 90 degrees
- moved J2 21.6 mm to (178.1, 105.2)
- moved J1 20.6 mm to (178.1, 89.5)
- moved R7 20.4 mm to (169.7, 107.1), turned to 90 degrees
- moved R6 20.4 mm to (171.2, 107.1), turned to 90 degrees
- moved U3 20.4 mm to (175.4, 98.0), turned to 180 degrees
- moved R13 20.3 mm to (160.8, 107.1), turned to 90 degrees
- moved R14 19.8 mm to (159.3, 107.1), turned to 90 degrees
- moved J6 19.8 mm to (153.5, 109.2)
- moved R16 18.2 mm to (156.3, 107.1), turned to 90 degrees
- moved R10 17.7 mm to (165.2, 107.1), turned to 90 degrees
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Connections:
- C9 pad 1: Net-(C9-Pad1) -> /vbus
- J2 pad 1: Net-(C9-Pad1) -> /vbus
- J4 pad 4: /i2c_sda -> /i2c_scl
- J4 pad 5: /i2c_scl -> /i2c_sda
- J5 pad 4: /spi_sck -> /spi_mosi
- J5 pad 6: /spi_mosi -> /spi_sck
- J6 pad 10: /pa6 -> /pb0
- J6 pad 11: /pa5 -> /pb1
- J6 pad 12: /pa4 -> /pb2
- J6 pad 13: /pc4 -> /pb10
- J6 pad 14: /pc5 -> /pb11
- J6 pad 4: /pb10 -> /pa4
- J6 pad 5: /pb11 -> /pa5
- J6 pad 6: /pb2 -> /pa6
- J6 pad 7: /pb1 -> /pa7
- J6 pad 8: /pb0 -> /pc4
- J6 pad 9: /pa7 -> /pc5
- R10 pad 1: /pa6 -> /pb0
- R11 pad 1: /pa7 -> /pc5
- R12 pad 1: /pb0 -> /pc4
- R13 pad 1: /pb1 -> /pa7
- R14 pad 1: /pb2 -> /pa6
- R15 pad 1: /pb11 -> /pa5
- R16 pad 1: /pb10 -> /pa4
- R6 pad 1: /pc5 -> /pb11
- R7 pad 1: /pc4 -> /pb10
- R8 pad 1: /pa4 -> /pb2
- R9 pad 1: /pa5 -> /pb1
Routing:
- net GND: track 165.4 -> 114.4 mm
- net /vbus: track 0.00 -> 38.9 mm
- net (no net): track 38.5 -> 0.00 mm, vias 2 -> 0
- net VDD: track 99.6 -> 88.3 mm
- net /i2c_sda: track 0.00 -> 11.3 mm
- net /i2c_scl: track 0.00 -> 10.8 mm
- net /spi_nss: track 0.00 -> 10.4 mm
- net /pb11: track 0.00 -> 10.3 mm
- net /pa4: track 0.00 -> 9.82 mm
- net /pb10: track 0.00 -> 9.61 mm
- net /spi_sck: track 0.00 -> 9.60 mm
- net /pa5: track 0.00 -> 9.15 mm
- net /pb2: track 0.00 -> 9.02 mm
- net /spi_miso: track 0.00 -> 8.69 mm
- net /pb1: track 0.00 -> 8.25 mm
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- removed copper zone on F.Cu, net GND
- removed copper zone on B.Cu, net VDD
Other:
- board outline removed

Commit message: Done with layout.
Routing:
- net VDD: track 88.3 -> 215.3 mm, vias 5 -> 9
- net GND: track 114.4 -> 219.3 mm
- net /vbus: track 38.9 -> 128.8 mm, vias 0 -> 1
- net /~mcu-rst~: track 2.86 -> 5.88 mm
- net /boot0: track 2.58 -> 4.48 mm
- added copper zone on B.Cu, net GND
- added copper zone on F.Cu, net GND
Other:
- board outline added: 39.5 x 32.5 mm
